File: hardware/kicad/esphome-smart-dimmer-1x1.kicad_pcb (KiCad board)
At the start: 2 copper layers, 30.8 x 47.8 mm, 9 parts, among them J1 USB_A, J2 USB_A, M3 MountingHole_3.2mm_M3, Q1 IRLB8721PBF, U1 ESP32-C3_SUPERMINI_TH

Commit message: Update esphome-smart-dimmer-1x1.kicad_pcb
Other:
- board text added: "ESPHome-Smart-Dimmer-1x1"
- board text removed: "Usb Light Dimmer Unit A"
